Commit message: fixed finray collision scaling

File: robot_filter/panda_description/urdf/panda_arm_hand_finray_wrist.urdf (robot description, URDF)
Before this commit: robot panda, 13 links, 12 joints
Links:
- link panda_leftfinger: geometry collision mesh filename=package://panda_description/meshes/collision/finger.stl scale=0.001 0.001 0.001; visual mesh filename=package://panda_description/meshes/visual/finray.dae scale=0.001 0.001 0.001
- link panda_rightfinger: geometry collision mesh filename=package://panda_description/meshes/collision/finger.stl scale=0.001 0.001 0.001; visual mesh filename=package://panda_description/meshes/visual/finray.dae scale=0.001 0.001 0.001

Commit message: reverted last commit

File: robot_filter/panda_description/urdf/panda_arm_hand_finray_wrist.urdf (robot description, URDF)
Before this commit: robot panda, 13 links, 12 joints
Links:
- link panda_leftfinger: geometry collision mesh filename=package://panda_description/meshes/collision/finger.stl; visual mesh filename=package://panda_description/meshes/visual/finray.dae scale=0.001 0.001 0.001
- link panda_rightfinger: geometry collision mesh filename=package://panda_description/meshes/collision/finger.stl; visual mesh filename=package://panda_description/meshes/visual/finray.dae scale=0.001 0.001 0.001
