Commit message: get gripper pcd in robotfilter

File: robot_filter/panda_description/urdf/panda_gripper_wrist.urdf (robot description, URDF)
Before this commit: robot panda_gripper, 4 links, 3 joints
Links:
- added link gripper_base, mass 0.001
- added link panda_wrist_cam_box, mass 0.05; collision box size=0.06 0.04 0.005; visual box size=0.06 0.04 0.005
- link panda_wrist_cam: mass 0.05 -> 0.03; geometry collision mesh filename=package://panda_description/meshes/collision/wrist_cam.stl scale=0.001 0.001 0.001; visual mesh filename=package://panda_description/meshes/visual/wrist_cam.dae scale=0.001 0.001 0.001
Joints:
- added joint gripper_base_to_hand: type fixed, parent gripper_base, child panda_hand, origin xyz=0 0 0 rpy=0 3.141593 3.141593
- added joint panda_wrist_cam_box_joint: type fixed, parent panda_hand, child panda_wrist_cam_box, origin xyz=-0.05 0 0.00 rpy=0 0 0
- joint panda_wrist_cam_joint: origin xyz=-0.05 0 0.00 rpy=0 0 0 -> xyz=-0.01 0 0.03 rpy=0 0 0; parent panda_hand -> panda_wrist_cam_box

Commit message: change to gripper rendering in traj loader and obs processor

File: robot_filter/panda_description/urdf/panda_gripper_wrist.urdf (robot description, URDF)
Before this commit: robot panda_gripper, 6 links, 5 joints
Joints:
- joint panda_finger_joint1: origin xyz=0 0 0.0584 rpy=0 0 0 -> xyz=0 0 0.0684 rpy=0 0 0
- joint panda_finger_joint2: origin xyz=0 0 0.0584 rpy=0 0 0 -> xyz=0 0 0.0684 rpy=0 0 0
